File: eagle-74hc595-led-test/led-test.sch (EAGLE design)
At the start: 38 parts, among them IC1 74HC595N, IC2 74HC595N, U1 PRO_MICRO_C

Commit message: added cap
Parts:
- added C4: (no value), gm-caps-film-box:072X0252
Connections:
- net GND: now also C4.2
- net N$1: now also C4.1
