File: eagle-74hc595-led-test/led-test.brd (EAGLE design)
At the start: 100 x 80 mm, 38 parts, among them IC1 74HC595N, IC2 74HC595N, U1 PRO_MICRO_C

Commit message: added cap
Parts:
- added C4: (no value), gm-caps-film-box:072X025
- moved C1 3.81 mm to (68.6, 67.3)
Connections:
- net GND: now also C4.2
- net N$1: now also C4.1
Routing:
- net GND: track 250.5 -> 256.8 mm
- net N$2: track 20.3 -> 25.4 mm

Commit message: updates
Routing:
- net N$4: track 26.7 -> 53.3 mm, vias 0 -> 4
- net N$1: track 25.4 -> 50.8 mm, vias 0 -> 3
- net N$39: track 24.1 -> 0.00 mm, vias 0 -> 1
- net N$38: track 24.1 -> 0.00 mm, vias 0 -> 1
- net N$6: track 11.4 -> 0.00 mm, vias 0 -> 1
- net N$22: track 7.62 -> 19.1 mm, vias 0 -> 2
- net N$2: track 25.4 -> 27.9 mm, vias 0 -> 1
- net N$7: track 25.4 -> 24.1 mm, vias 0 -> 1
- net GND: track 256.8 -> 258.1 mm, vias 0 -> 1
- net N$9: vias 0 -> 1
- net N$8: vias 0 -> 1
- net N$5: vias 0 -> 1
- net N$41: vias 0 -> 1
- net N$40: vias 0 -> 3
- net N$37: vias 0 -> 1
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
Commit message: eagle led updates
Routing:
- net GND: track 258.1 -> 265.7 mm, vias 1 -> 2
- net N$40: track 179.1 -> 184.2 mm
Changed lines of the file:
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@@
 <layer number="1" name="Top" color="4" fill="1" visible="no" active="yes"/>
 <layer number="16" name="Bottom" color="1" fill="1" visible="yes" active="yes"/>
-<layer number="17" name="Pads" color="2" fill="1" visible="yes" active="yes"/>
+<layer number="17" name="Pads" color="2" fill="1" visible="no" active="yes"/>
 <layer number="18" name="Vias" color="2" fill="1" visible="yes" active="yes"/>
 <layer number="19" name="Unrouted" color="6" fill="1" visible="no" active="yes"/>
-<layer number="20" name="Dimension" color="15" fill="1" visible="no" active="yes"/>
+<layer number="20" name="Dimension" color="15" fill="1" visible="yes" active="yes"/>
 <layer number="21" name="tPlace" color="7" fill="1" visible="yes" active="yes"/>
 <layer number="22" name="bPlace" color="7" fill="1" visible="yes" active="yes"/>
@@
 <circle x="58.42" y="54.61" radius="0.635" width="0.8128" layer="16"/>
 <circle x="58.42" y="43.18" radius="0.635" width="0.8128" layer="16"/>
-<rectangle x1="78.74" y1="27.94" x2="95.25" y2="39.37" layer="16"/>
-<rectangle x1="86.36" y1="38.1" x2="95.25" y2="44.45" layer="16"/>
-<rectangle x1="95.25" y1="27.94" x2="99.06" y2="72.39" layer="16"/>
 <rectangle x1="25.4" y1="27.94" x2="50.8" y2="30.48" layer="16"/>
 <rectangle x1="25.4" y1="52.07" x2="52.07" y2="54.61" layer="16"/>
@@
 <rectangle x1="57.15" y1="27.94" x2="80.01" y2="30.48" layer="16"/>
 <rectangle x1="72.39" y1="35.56" x2="80.01" y2="39.37" layer="16"/>
-<rectangle x1="95.25" y1="71.12" x2="99.06" y2="78.74" layer="16"/>
 </plain>
 <attributes>
@@
 <wire x1="67.31" y1="52.07" x2="67.31" y2="39.37" width="0.8128" layer="16"/>
 <wire x1="67.31" y1="39.37" x2="80.01" y2="39.37" width="0.8128" layer="16"/>
-<wire x1="80.01" y1="39.37" x2="95.25" y2="39.37" width="0.8128" layer="16"/>
-<wire x1="95.25" y1="39.37" x2="95.25" y2="72.39" width="0.8128" layer="16"/>
+<wire x1="80.01" y1="39.37" x2="99.06" y2="39.37" width="0.8128" layer="16"/>
+<wire x1="99.06" y1="39.37" x2="99.06" y2="72.39" width="0.8128" layer="16"/>
+<wire x1="99.06" y1="72.39" x2="95.25" y2="72.39" width="0.8128" layer="16"/>
 <wire x1="95.25" y1="72.39" x2="90.17" y2="72.39" width="0.8128" layer="16"/>
 <wire x1="50.8" y1="54.61" x2="50.8" y2="64.77" width="0.8128" layer="16"/>
@@
 <wire x1="63.5" y1="64.77" x2="63.5" y2="67.31" width="1.016" layer="16"/>
 <via x="90.17" y="72.39" extent="1-16" drill="0.35"/>
+<via x="95.25" y="72.39" extent="1-16" drill="0.35"/>
 <wire x1="90.17" y1="72.39" x2="91.44" y2="72.39" width="0" layer="19" extent="1-1"/>
 <wire x1="74.93" y1="30.75" x2="74.93" y2="30.48" width="0" layer="19" extent="16-16"/>
@@
 <wire x1="69.85" y1="41.91" x2="83.82" y2="41.91" width="0.8128" layer="16"/>
 <wire x1="83.82" y1="41.91" x2="83.82" y2="67.31" width="0.8128" layer="16"/>
-<wire x1="83.82" y1="67.31" x2="90.17" y2="67.31" width="0.8128" layer="16"/>
+<wire x1="83.82" y1="67.31" x2="95.25" y2="67.31" width="0.8128" layer="16"/>
 <wire x1="83.82" y1="77.47" x2="83.82" y2="67.31" width="0.8128" layer="16"/>
 <wire x1="54.61" y1="72.39" x2="68.58" y2="72.39" width="0.8128" layer="16"/>
@@
 <contactref element="C3" pad="+"/>
 <wire x1="65.405" y1="33.02" x2="74.93" y2="33.02" width="0.8128" layer="16"/>
-<via x="90.17" y="67.31" extent="1-16" drill="0.35"/>
+<via x="95.25" y="67.31" extent="1-16" drill="0.35"/>
 <via x="69.85" y="36.83" extent="1-16" drill="0.35"/>
 <via x="69.85" y="41.91" extent="1-16" drill="0.35"/>
-<wire x1="90.17" y1="67.31" x2="91.44" y2="67.31" width="0" layer="19" extent="1-1"/>
 <wire x1="74.93" y1="32.75" x2="74.93" y2="33.02" width="0" layer="19" extent="16-16"/>
+<wire x1="91.44" y1="67.31" x2="95.25" y2="67.31" width="0" layer="19"/>
 </signal>
 <signal name="N$3">
@@
 <via x="90.17" y="74.93" extent="1-16" drill="0.35"/>
 </signal>
+<signal name="N$57">
+<via x="95.25" y="74.93" extent="1-16" drill="0.35"/>
+</signal>
+<signal name="N$58">
+<via x="95.25" y="69.85" extent="1-16" drill="0.35"/>
+</signal>
+<signal name="N$59">
+<via x="90.17" y="67.31" extent="1-16" drill="0.35"/>
+</signal>
+<signal name="N$60">
+<via x="95.25" y="64.77" extent="1-16" drill="0.35"/>
+</signal>
+<signal name="N$61">
+<via x="95.25" y="62.23" extent="1-16" drill="0.35"/>
+</signal>
+<signal name="N$62">
+<via x="95.25" y="59.69" extent="1-16" drill="0.35"/>
+</signal>
+<signal name="N$63">
+<via x="95.25" y="57.15" extent="1-16" drill="0.35"/>
+</signal>
+<signal name="N$64">
+<via x="95.25" y="54.61" extent="1-16" drill="0.35"/>
+</signal>
+<signal name="N$65">
+<via x="95.25" y="46.99" extent="1-16" drill="0.35"/>
+</signal>
+<signal name="N$66">
+<via x="95.25" y="52.07" extent="1-16" drill="0.35"/>
+</signal>
+<signal name="N$67">
+<via x="95.25" y="49.53" extent="1-16" drill="0.35"/>
+</signal>
 </signals>
